File: Group 12.brd (EAGLE design)
At the start: 160 x 100 mm, 30 parts, among them U1 328P, Y1 16MHz

Commit message: board and sch
board and sch
Parts:
- removed U$1: USB-PWR, adafruit:USB-MINIB-THM-MOLEX-PWRONLY
- added C12: 100n, rcl:C0805K
- added ICSP: (no value), pinhead:2X03
- added J1: 6_PIN_SERIAL_CABLEPTH, SparkFun-Connectors:FTDI_BASIC
- added R10, R8, R9: 10k, rcl:R0805
- added R7: 220, rcl:R0805
- moved C10 51.5 mm to (61.7, 92.7), turned to 270 degrees
- moved S2 42.4 mm to (66.0, 45.0)
- moved S3 22.7 mm to (58.4, 26.2), turned to 0 degrees
- moved C7 14.1 mm to (69.3, 39.1)
- moved S4 10.9 mm to (77.5, 84.1)
- moved C8 8.87 mm to (65.3, 33.8), turned to 0 degrees
- moved Y1 8.40 mm to (70.9, 35.1)
- moved R6 7.13 mm to (100.3, 80.8)
Connections:
- removed net PD4: S2.2, U1.6
- removed net PD7: S3.2, U1.13
- new net CAL: R9.1, S2.2, U1.6
- new net MISO: ICSP.1, U1.18
- new net N$3: J1.RXI, U1.3
- new net N$4: ICSP.4, U1.17
- new net SCK: ICSP.3, U1.19
- new net SET: R8.1, S3.2, U1.13
- net 5V: now also C12.1, ICSP.2, J1.VCC, R10.1, R8.2, R9.2; no longer U$1.VBUS
- net GND: now also 74HC132.11, 74HC132.12, 74HC132.13, C12.2, ICSP.6, J1.GND, R7.2; no longer U$1.GND
- net PD0: now also J1.TXO, R10.2, R7.1
- net RESET: now also ICSP.5
Routing:
- net 5V: track 261.5 -> 319.0 mm, vias 8 -> 13
- net N$3: track 0.00 -> 57.2 mm, vias 0 -> 1
- net PD4: track 52.7 -> 0.00 mm
- net SCK: track 0.00 -> 47.7 mm, vias 0 -> 2
- net PD0: track 22.5 -> 65.0 mm, vias 0 -> 1
- net PD7: track 41.6 -> 0.00 mm
- net RESET: track 62.2 -> 99.2 mm, vias 1 -> 4
- net MISO: track 0.00 -> 34.1 mm, vias 0 -> 1
- net N$4: track 0.00 -> 30.8 mm, vias 0 -> 2
- net SET: track 0.00 -> 25.9 mm, vias 0 -> 2
- net PB6: track 27.3 -> 8.01 mm, vias 2 -> 0
- net CAL: track 0.00 -> 11.2 mm
- net PB7: track 21.0 -> 12.7 mm, vias 0 -> 2
- net N$22: track 33.9 -> 41.6 mm
Other:
- board text added: "Team 12"
- board text added: "Version: 5.0"

Commit message: final sch and brd
final sch and brd
Parts:
- removed 74HC132: 4093D, adafruit:SO14
- removed C0003: 100n, rcl:C0805K
- removed TP1, TP2, TP3, TP4, TP5, TP6, TP7, TP8: TPPAD1-13, testpad:P1-13
- added C13: 100n, rcl:C0805K
- added C14: .1u, rcl:C0805K
- added CAP, IND, RES: (no value), pinhead:1X02
- added IC1: 74LS132D, 74xx-us:SO14
- added L1: 1m, rcl:0204/5
- R7: value 220 -> 10k
- moved C6 96.8 mm to (22.6, 42.4), turned to 180 degrees
- moved C0048 79.8 mm to (59.9, 54.4)
- moved C1 68.2 mm to (29.0, 17.5), turned to 0 degrees
- moved R6 67.7 mm to (35.6, 61.2)
- moved R1 66.9 mm to (30.2, 60.5), turned to 90 degrees
- moved ICSP 65.5 mm to (37.8, 29.5)
- moved R2 64.1 mm to (40.6, 8.38)
- moved J1 57.8 mm to (21.6, 64.8)
- moved C10 57.6 mm to (13.5, 61.2), turned to 180 degrees
- moved R9 56.3 mm to (16.8, 42.9), turned to 270 degrees
- moved S4 56.0 mm to (25.4, 63.5)
- moved R5 53.3 mm to (32.5, 11.7), turned to 180 degrees
- moved S2 52.7 mm to (14.2, 54.4), turned to 270 degrees
- moved U1 50.8 mm to (29.5, 39.1)
- moved R8 50.3 mm to (21.8, 16.5), turned to 270 degrees
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Connections:
- new net MODE: R10.2, S1.2, U1.5
- new net N$7: C14.1, J1.DTR
- net 5V: now also C13.1, IC1.14; no longer 74HC132.14, C0003.1
- net GND: now also C13.2, CAP.1, IC1.12, IC1.13, IC1.7; no longer 74HC132.11, 74HC132.12, 74HC132.13, 74HC132.7, C0003.2, TP8.TP
- net N$1: now also C2.1, CAP.2, IC1.1, R3.2; no longer 74HC132.9, R4.1
- net N$10: now also IC1.5, IC1.8, L1.2; no longer 74HC132.10, 74HC132.6, TP1.TP
- net N$14: now also IND.1, L1.1; no longer TP2.TP, TP6.TP
- net N$16: now also IND.2, RES.2; no longer TP3.TP, TP4.TP
- net N$17: now also RES.1; no longer TP5.TP
- net N$2: now also IC1.10, R4.1; no longer 74HC132.1, C2.1, R3.2, TP7.TP
- net N$5: now also IC1.3, IC1.4; no longer 74HC132.3, 74HC132.5
- net PD0: no longer R10.2, S1.2
- net PD2: now also IC1.2; no longer 74HC132.2
- net PD5: now also IC1.6; no longer 74HC132.4
- net PD6: now also IC1.9; no longer 74HC132.8
- net RESET: now also C14.2
Routing:
- net 5V: track 319.0 -> 182.4 mm, vias 13 -> 8
- net RESET: track 99.2 -> 43.5 mm, vias 4 -> 3
- net PD5: track 74.0 -> 19.4 mm, vias 4 -> 0
- net PD0: track 65.0 -> 17.9 mm
- net N$7: track 0.00 -> 42.8 mm, vias 0 -> 2
- net N$2: track 52.5 -> 12.0 mm, vias 1 -> 0
- net SCK: track 47.7 -> 7.21 mm, vias 2 -> 0
- net N$3: track 57.2 -> 22.3 mm
- net N$22: track 41.6 -> 8.25 mm, vias 1 -> 0
- net PC4: track 41.4 -> 11.3 mm
- net PC3: track 40.1 -> 11.3 mm
- net PC2: track 40.1 -> 11.3 mm
- net PC5: track 40.1 -> 11.4 mm
- net PC0: track 48.7 -> 20.4 mm
- net MISO: track 34.1 -> 7.21 mm, vias 1 -> 0
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Other:
- board size 160 x 100 mm -> 47.2 x 69.1 mm

Commit message: final brd and sch
final brd and sch
Parts:
- added TP1, TP10, TP11, TP12, TP13, TP14, TP15, TP16, TP17, TP18, TP19, TP2, TP20, TP21, TP22, TP23, TP24, TP25, TP26, TP27, TP28, TP29, TP3, TP30, TP31, TP4, TP5, TP6, TP7, TP8, TP9: TPPAD1-13, testpad:P1-13
Connections:
- removed net N$17: R5.2, RES.1
- new net N$8: R5.2, RES.1, TP29.TP
- net 5V: now also TP22.TP
- net CAL: now also TP24.TP
- net GND: now also TP9.TP
- net MISO: now also TP11.TP
- net MODE: now also TP23.TP
- net N$1: now also TP15.TP, TP31.TP
- net N$10: now also TP1.TP
- net N$14: now also TP30.TP
- net N$16: now also TP28.TP
- net N$2: now also TP18.TP
- net N$3: now also TP20.TP
- net N$4: now also TP10.TP
- net N$5: now also TP14.TP
- net N$7: now also TP19.TP
- net PB6: now also TP26.TP
- net PB7: now also TP27.TP
- net PC0: now also TP3.TP
- net PC1: now also TP4.TP
- net PC2: now also TP5.TP
- net PC3: now also TP6.TP
- net PC4: now also TP7.TP
- net PC5: now also TP8.TP
- net PD0: now also TP21.TP
- net PD2: now also TP16.TP
- net PD5: now also TP2.TP
- net PD6: now also TP17.TP
- net RESET: now also TP13.TP
- net SCK: now also TP12.TP
- net SET: now also TP25.TP
Routing:
- net PC2: track 11.3 -> 29.7 mm, vias 0 -> 1
- net PC3: track 11.3 -> 27.9 mm, vias 0 -> 1
- net PC4: track 11.3 -> 26.7 mm, vias 0 -> 1
- net MISO: track 7.21 -> 17.3 mm
- net 5V: track 182.4 -> 192.0 mm
- net N$8: track 0.00 -> 9.52 mm
- net N$1: track 39.2 -> 47.3 mm
- net N$4: track 4.04 -> 10.8 mm
- net N$17: track 5.75 -> 0.00 mm
- net CAL: track 20.1 -> 25.1 mm
- net N$10: track 56.5 -> 61.4 mm
- net N$5: track 13.2 -> 18.1 mm
- net MODE: track 11.7 -> 16.5 mm
- net PC0: track 20.4 -> 25.1 mm
- net PD6: track 29.8 -> 33.7 mm
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