File: Group 12.sch (EAGLE design)
At the start: 13 parts

Commit message: Schm and Proj Sch
Schematic and Project Schedule
Parts:
- removed L1: 1m, rcl:L-USL1812
- removed SWITCH1, SWITCH2, SWITCH3: MOMENTARY-SWITCH-SPST-SMD-6.0X3.5MM, SparkFun-Switches:MOMENTARY-SWITCH-SPST-SMD-6.0X3.5MM
- removed U$1: ARDUINOUNO, adafruit:ARDUINOUNO
- added C0003, C0004, C6: 100n, rcl:C-EUC0805K
- added C7, C8: 22p, rcl:C-EUC0805K
- added JP2: (no value), pinhead:PINHD-1X8
- added R2: 20k, rcl:POTENTIOMETER_PT-10
- added R6: 220, rcl:R-US_R0805
- added S1, S2, S3, S4: MOMENTARY-SWITCH-SPST-SMD-6.0X3.5MM, SparkFun-Switches:MOMENTARY-SWITCH-SPST-SMD-6.0X3.5MM
- added TP1, TP2, TP3, TP4, TP5, TP6, TP7, TP8: TPPAD1-13, testpad:TPPAD1-13
- added U1: 328P, SparkFun-IC-Microcontroller:ATMEGA328P_PDIP
- added Y1: 16MHz, SparkFun-Clocks:CRYSTAL-16MHZSMD-5X3.2
- R1: value 20k -> 10k; device rcl:POTENTIOMETER_PT_SPIN -> rcl:R-US_R0805
Connections:
- removed net N$19: SWITCH3.2, U$1.D7
- new net N$22: C0048.K, R6.2
- new net N$24: C7.2, U1.PB6(XTAL1/TOSC1), Y1.2
- new net N$25: C8.2, U1.PB7(XTAL2/TOSC2), Y1.1
- new net N$35: 74HC132C.O, JP2.6, U1.PD5(T1)
- new net N$36: JP2.4, U1.PD3(INT1)
- new net N$37: JP2.5, S2.2
- new net N$39: JP2.2, U1.PD1(TXD)
- new net N$40: JP2.1, S1.2, U1.PD0(RXD)
- net 5V: now also C0003.1, C0004.1, C0048.VDD, C6.1, R1.2, R2.2, R6.1, U1.AVCC, U1.VCC; no longer 74HC132D.I0, 74HC132D.I1, C0048.A
- net GND: now also C0003.2, C0004.2, C0048.A, C6.2, C7.1, C8.1, R2.1, S1.1, S2.1, S3.1, S4.1, TP8.TP, U1.GND@1, U1.GND@2; no longer C0048.K, R1.1, SWITCH1.1, SWITCH2.1, SWITCH3.1, U$1.GND, U$1.GND1, U$1.GND2
- net N$1: now also JP2.8, S3.2; no longer SWITCH1.2, U$1.D0
- net N$10: no longer L1.2
- net N$12: now also TP4.TP
- net N$13: now also TP1.TP; no longer 74HC132C.O, U$1.D5
- net N$14: now also TP2.TP, TP6.TP; no longer 74HC132B.I0, U$1.D6
- net N$15: now also R1.1, S4.2, U1.PC6(/RESET); no longer 74HC132A.I1, U$1.D2
- net N$16: now also TP3.TP; no longer L1.1
- net N$17: now also TP5.TP
- net N$18: now also 74HC132B.I0, JP2.7, U1.PD6(AIN0); no longer SWITCH2.2, U$1.D4
- net N$2: now also TP7.TP
- net N$20: now also R2.3; no longer R1.3
- net N$21: now also U1.PC0(ADC0); no longer U$1.A0
- net N$3: now also 74HC132A.I1, JP2.3, U1.PD2(INT0); no longer C0048.VDD, R1.2, U$1.5V
- net N$4: now also U1.PC1(ADC1); no longer U$1.A1
- net N$5: now also U1.PC2(ADC2); no longer U$1.A2
- net N$6: now also U1.PC3(ADC3); no longer U$1.A3
- net N$7: now also U1.PC4(ADC4/SDA); no longer U$1.A4
- net N$8: now also U1.PC5(ADC5/SCL); no longer U$1.A5
Other:
- note added: "D0"
- note added: "D1"
- note added: "D2"
- note added: "D3"
- note added: "D4"
- note added: "D5"
- note added: "D6"
- note added: "D7"
- moved on the sheet: 74HC132A, 74HC132B, 74HC132C, 74HC132P, C0048, C1, C2, R3, R4, R5

Commit message: Final Schem
Final Schem
Other:
- note added: "11/1/17"
- note added: "2.0"
- note removed: "1.0"
- note removed: "10/25/17"
Changed lines of the file:
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@@
 <text x="19.304" y="56.388" size="1.778" layer="97">Cx</text>
 <text x="21.844" y="28.448" size="1.778" layer="97">Lx</text>
-<text x="184.15" y="1.27" size="1.778" layer="95">10/25/17</text>
+<text x="184.15" y="1.27" size="1.778" layer="95">11/1/17</text>
 <text x="205.74" y="8.89" size="1.778" layer="95">ECE 411 GROUP 12 SCHEMATIC</text>
-<text x="265.43" y="7.62" size="1.778" layer="95">1.0</text>
+<text x="265.43" y="7.62" size="1.778" layer="95">2.0</text>
 <text x="238.76" y="104.14" size="1.778" layer="97">D7</text>
 <text x="238.76" y="106.68" size="1.778" layer="97">D6</text>

Commit message: board and sch
board and sch
Parts:
- removed C0004: 100n, rcl:C-EUC0805K
- removed JP2: (no value), pinhead:PINHD-1X8
- added C10: 4.7u, rcl:C-EUC0805K
- added C12: 100n, rcl:C-EUC0805K
- added ICSP: (no value), pinhead:PINHD-2X3
- added J1: 6_PIN_SERIAL_CABLEPTH, SparkFun-Connectors:6_PIN_SERIAL_CABLEPTH
- added R10, R8, R9: 10k, rcl:R-US_R0805
- added R7: 220, rcl:R-US_R0805
Connections:
- net N$21 renamed PC0
- net N$24 renamed PB6
- net N$25 renamed PB7
- net N$4 renamed PC1
- net N$5 renamed PC2
- net N$6 renamed PC3
- net N$7 renamed PC4
- net N$8 renamed PC5
- removed net N$11: 74HC132B.I1, R4.1
- removed net N$12: C1.1, R4.2, TP4.TP
- removed net N$13: TP1.TP
- removed net N$15: R1.1, S4.2, U1.PC6(/RESET)
- removed net N$18: 74HC132B.I0, JP2.7, U1.PD6(AIN0)
- removed net N$35: 74HC132C.O, JP2.6, U1.PD5(T1)
- removed net N$36: JP2.4, U1.PD3(INT1)
- removed net N$37: JP2.5, S2.2
- removed net N$39: JP2.2, U1.PD1(TXD)
- removed net N$40: JP2.1, S1.2, U1.PD0(RXD)
- removed net N$9: 74HC132A.O, 74HC132C.I0, R3.1
- new net CAL: R9.1, S2.2, U1.PD4(XCK/T0)
- new net MISO: ICSP.1, U1.PB4(MISO)
- new net N$4: ICSP.4, U1.PB3(MOSI/OC2)
- new net N$5: 74HC132A.O, 74HC132B.I0, R3.1
- new net PD0: J1.3, R10.2, R7.1, S1.2, U1.PD0(RXD)
- new net PD2: 74HC132A.I1, U1.PD2(INT0)
- new net PD5: 74HC132B.O, U1.PD5(T1)
- new net PD6: 74HC132C.I0, U1.PD6(AIN0)
- new net RESET: ICSP.5, R1.1, S4.2, U1.PC6(/RESET)
- new net SCK: ICSP.3, U1.PB5(SCK)
- new net SET: R8.1, S3.2, U1.PD7(AIN1)
- net 5V: now also C10.1, C12.1, ICSP.2, J1.4, R10.1, R8.2, R9.2; no longer C0004.1
- net GND: now also 74HC132D.I0, 74HC132D.I1, 74HC132D.O, C10.2, C12.2, ICSP.6, J1.6, R7.2; no longer C0004.2
- net N$1: now also 74HC132C.I1, R4.1; no longer JP2.8, S3.2
- net N$10: now also 74HC132B.I1, 74HC132C.O, TP1.TP; no longer 74HC132B.O, 74HC132C.I1
- net N$16: now also C1.1, R4.2, TP4.TP
- net N$3: now also J1.2, U1.PD1(TXD); no longer 74HC132A.I1, JP2.3, U1.PD2(INT0)
Other:
- note added: "5.0"
- note added: "ATMEGA CHIP FROM ARDUINO AND ICSP"
- note added: "Inductor"
- note added: "LCD SCREEN DISPLAYS COMPONENT VALUE"
- note added: "LCR Meter"
- note added: "POWER"
- note added: "SCHMITT NAND GATE"
- note removed: "2.0"
- note removed: "D0"
- note removed: "D1"
- note removed: "D2"
- note removed: "D3"
- note removed: "D4"
- note removed: "D5"
- note removed: "D6"
- note removed: "D7"
- moved on the sheet: 74HC132A, 74HC132B, 74HC132C, C0003, C1, C2, R3, R4, R5, S1, S2, S3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

Commit message: final sch and brd
final sch and brd
Parts:
- removed 74HC132: 4093D, adafruit:4093D
- removed C0003: 100n, rcl:C-EUC0805K
- removed TP1, TP2, TP3, TP4, TP5, TP6, TP7, TP8: TPPAD1-13, testpad:TPPAD1-13
- added C13: 100n, rcl:C-EUC0805K
- added C14: .1u, rcl:C-EUC0805K
- added CAP, IND, RES: (no value), pinhead:PINHD-1X2
- added IC1: 74LS132D, 74xx-us:74LS132D
- added L1: 1m, rcl:L-US0204/5
- R7: value 220 -> 10k
Connections:
- new net MODE: R10.2, S1.2, U1.PD3(INT1)
- new net N$7: C14.1, J1.1
- net 5V: now also C13.1, IC1P.VCC; no longer 74HC132P.VDD, C0003.1
- net GND: now also C13.2, CAP.1, IC1D.I0, IC1D.I1, IC1P.GND; no longer 74HC132D.I0, 74HC132D.I1, 74HC132D.O, 74HC132P.VSS, C0003.2, TP8.TP
- net N$1: now also C2.1, CAP.2, IC1A.I0, R3.2; no longer 74HC132C.I1, R4.1
- net N$10: now also IC1B.I1, IC1C.O, L1.2; no longer 74HC132B.I1, 74HC132C.O, TP1.TP
- net N$14: now also IND.1, L1.1; no longer TP2.TP, TP6.TP
- net N$16: now also IND.2, RES.2; no longer TP3.TP, TP4.TP
- net N$17: now also RES.1; no longer TP5.TP
- net N$2: now also IC1C.I1, R4.1; no longer 74HC132A.I0, C2.1, R3.2, TP7.TP
- net N$5: now also IC1A.O, IC1B.I0; no longer 74HC132A.O, 74HC132B.I0
- net PD0: no longer R10.2, S1.2
- net PD2: now also IC1A.I1; no longer 74HC132A.I1
- net PD5: now also IC1B.O; no longer 74HC132B.O
- net PD6: now also IC1C.I0; no longer 74HC132C.I0
- net RESET: now also C14.2
Other:
- note removed: "Cx"
- note removed: "Inductor"
- note removed: "Lx"
- note removed: "Rx"
- moved on the sheet: C1, C10, C12, C2, C6, C7, C8, R3, R4

Commit message: final brd and sch
final brd and sch
Parts:
- added TP1, TP10, TP11, TP12, TP13, TP14, TP15, TP16, TP17, TP18, TP19, TP2, TP20, TP21, TP22, TP23, TP24, TP25, TP26, TP27, TP28, TP29, TP3, TP30, TP31, TP4, TP5, TP6, TP7, TP8, TP9: TPPAD1-13, testpad:TPPAD1-13
Connections:
- removed net N$17: R5.2, RES.1
- new net N$8: R5.2, RES.1, TP29.TP
- net 5V: now also TP22.TP
- net CAL: now also TP24.TP
- net GND: now also TP9.TP
- net MISO: now also TP11.TP
- net MODE: now also TP23.TP
- net N$1: now also TP15.TP, TP31.TP
- net N$10: now also TP1.TP
- net N$14: now also TP30.TP
- net N$16: now also TP28.TP
- net N$2: now also TP18.TP
- net N$3: now also TP20.TP
- net N$4: now also TP10.TP
- net N$5: now also TP14.TP
- net N$7: now also TP19.TP
- net PB6: now also TP26.TP
- net PB7: now also TP27.TP
- net PC0: now also TP3.TP
- net PC1: now also TP4.TP
- net PC2: now also TP5.TP
- net PC3: now also TP6.TP
- net PC4: now also TP7.TP
- net PC5: now also TP8.TP
- net PD0: now also TP21.TP
- net PD2: now also TP16.TP
- net PD5: now also TP2.TP
- net PD6: now also TP17.TP
- net RESET: now also TP13.TP
- net SCK: now also TP12.TP
- net SET: now also TP25.TP
Other:
- moved on the sheet: R5
